File: data/templates/active-lpf-sallen-key/{{PROJECT_NAME}}.kicad_sch (KiCad schematic)
At the start: 7 parts, among them U1 TL072

Commit message: T029 Phase 0: fix 4 dirty templates via builders
Builders (active-lpf-sallen-key, op-amp-inverting, bjt-ce-nfb) add a
PWR_FLAG on the GND net to clear ERC `power_pin_not_driven`. The
tube-line-preamp builder fixes r_g2.pin_b wiring — previous connect
target (114.3, 90.17) was the pin's own coordinate (zero-length wire),
leaving R4 pin 1 floating; new target (114.3, 88.9) places it on the
grid2 net as a canonical grid-leak.

data/templates/* regenerated via scripts/regenerate-templates.py. All
11 templates now ERC-clean (errors=0) — satisfies T029 SC1.

Calibration baselines for tube-line-preamp updated to reflect the now
correctly-biased CF: V_cathode2 window 30-150V → 2-50V; mid-band gain
baseline 64.0 → 54.0 V/V (matches analytical 54 V/V hand-calc exactly,
which is now achievable because R4 grid-leak loads C3→V1B coupling per
hand-calc assumption).

Spec §6 A1 amended: fix path is "via builders + regen", not direct
edits to data/templates/. Direct-edit probe (2026-06-05) confirmed
0-errors achievable but breaks snapshot tests and is wiped by next
regenerate-templates.py.

Pre-push 5/5 ✓ (ruff/format/mypy clean; 2025 passed, 10 skipped,
1 xfailed; coverage 86.98%).

Co-Authored-By: Claude Opus 4.7 (1M context) <noreply@anthropic.com>
Changed lines of the file:
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@@
+	(wire
+		(pts
+			(xy 44.92 78.74) (xy 50 78.74)
+		)
+		(stroke
+			(width 0)
+			(type default)
+		)
+	)
 	(wire
 		(pts
@@
 					(unit 1)
 				)
+			)
+		)
+	)
+	(symbol
+		(lib_id "power:PWR_FLAG")
+		(at 44.92 78.74 180)
+		(unit 1)
+		(body_style 1)
+		(exclude_from_sim no)
+		(in_bom yes)
+		(on_board yes)
+		(in_pos_files yes)
+		(dnp no)
+		(fields_autoplaced yes)
+		(property "Reference" "#FLG01"
+			(at 44.92 76.84 0)
+			(hide yes)
+			(show_name no)
+			(do_not_autoplace no)
+			(effects
+				(font
+					(size 1.27 1.27)
+				)
+			)
+		)
+		(property "Value" "PWR_FLAG"
+			(at 44.92 84.84 0)
+			(show_name no)
+			(do_not_autoplace no)
+			(effects
+				(font
+					(size 1.27 1.27)
+				)
+			)
+		)
+		(property "Footprint" ""
+			(at 44.92 78.74 0)
+			(show_name no)
+			(do_not_autoplace no)
+			(effects
+				(font
+					(size 1.27 1.27)
+				)
+			)
+		)
+		(property "Datasheet" ""
+			(at 44.92 78.74 0)
+			(show_name no)
+			(do_not_autoplace no)
+			(effects
+				(font
+					(size 1.27 1.27)
+				)
+			)
+		)
+		(property "Description" ""
+			(at 44.92 78.74 0)
+			(hide yes)
+			(show_name no)
+			(do_not_autoplace no)
+			(effects
+				(font
+					(size 1.27 1.27)
+				)
+			)
+		)
+		(pin "1"
+		)
+		(instances
+			(project "active_lpf_sallen_key"
+				(path "/d845d22c-4ed8-40fd-884e-d999f7ab0ead"
+					(reference "#FLG01")
+					(unit 1)
+				)
