File: data/templates/op-amp-inverting/{{PROJECT_NAME}}.kicad_sch (KiCad schematic)
At the start: 5 parts, among them U1 GENERIC_OPAMP_2POLE

Commit message: T029 Phase 0: fix 4 dirty templates via builders
Builders (active-lpf-sallen-key, op-amp-inverting, bjt-ce-nfb) add a
PWR_FLAG on the GND net to clear ERC `power_pin_not_driven`. The
tube-line-preamp builder fixes r_g2.pin_b wiring — previous connect
target (114.3, 90.17) was the pin's own coordinate (zero-length wire),
leaving R4 pin 1 floating; new target (114.3, 88.9) places it on the
grid2 net as a canonical grid-leak.

data/templates/* regenerated via scripts/regenerate-templates.py. All
11 templates now ERC-clean (errors=0) — satisfies T029 SC1.

Calibration baselines for tube-line-preamp updated to reflect the now
correctly-biased CF: V_cathode2 window 30-150V → 2-50V; mid-band gain
baseline 64.0 → 54.0 V/V (matches analytical 54 V/V hand-calc exactly,
which is now achievable because R4 grid-leak loads C3→V1B coupling per
hand-calc assumption).

Spec §6 A1 amended: fix path is "via builders + regen", not direct
edits to data/templates/. Direct-edit probe (2026-06-05) confirmed
0-errors achievable but breaks snapshot tests and is wiped by next
regenerate-templates.py.

Pre-push 5/5 ✓ (ruff/format/mypy clean; 2025 passed, 10 skipped,
1 xfailed; coverage 86.98%).

Co-Authored-By: Claude Opus 4.7 (1M context) <noreply@anthropic.com>
Parts:
- removed R_fb: 10k, symbol Device:R
- added R_load: 1Meg, symbol Device:R
- R_fb: renamed from R_load; value 1Meg -> 10k
Connections:
- net GND: now also R_load.2; no longer R_fb.2
- net in_neg: now also R_fb.1
- net vout: now also R_fb.2, R_load.1; no longer R_fb.1
Other:
- moved on the sheet: R_fb
Changed lines of the file:
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@@
+	(wire
+		(pts
+			(xy 77.3 67.31) (xy 82.38 67.31)
+		)
+		(stroke
+			(width 0)
+			(type default)
+		)
+	)
 	(wire
 		(pts
@@
 					(unit 1)
 				)
+			)
+		)
+	)
+	(symbol
+		(lib_id "power:PWR_FLAG")
+		(at 77.3 67.31 180)
+		(unit 1)
+		(body_style 1)
+		(exclude_from_sim no)
+		(in_bom yes)
+		(on_board yes)
+		(in_pos_files yes)
+		(dnp no)
+		(fields_autoplaced yes)
+		(property "Reference" "#FLG01"
+			(at 77.3 65.41 0)
+			(hide yes)
+			(show_name no)
+			(do_not_autoplace no)
+			(effects
+				(font
+					(size 1.27 1.27)
+				)
+			)
+		)
+		(property "Value" "PWR_FLAG"
+			(at 77.3 73.41 0)
+			(show_name no)
+			(do_not_autoplace no)
+			(effects
+				(font
+					(size 1.27 1.27)
+				)
+			)
+		)
+		(property "Footprint" ""
+			(at 77.3 67.31 0)
+			(show_name no)
+			(do_not_autoplace no)
+			(effects
+				(font
+					(size 1.27 1.27)
+				)
+			)
+		)
+		(property "Datasheet" ""
+			(at 77.3 67.31 0)
+			(show_name no)
+			(do_not_autoplace no)
+			(effects
+				(font
+					(size 1.27 1.27)
+				)
+			)
+		)
+		(property "Description" ""
+			(at 77.3 67.31 0)
+			(hide yes)
+			(show_name no)
+			(do_not_autoplace no)
+			(effects
+				(font
+					(size 1.27 1.27)
+				)
+			)
+		)
+		(pin "1"
+		)
+		(instances
+			(project "op_amp_inverting"
+				(path "/af8fa3e2-64a9-4760-bd01-db445500be86"
+					(reference "#FLG01")
+					(unit 1)
+				)
